File: SATA_board/SATA_board.kicad_pcb (KiCad board)
At the start: 4 copper layers, 120 x 60.5 mm, 212 parts, among them J1 105310-1206, J2 USB_C_Receptacle_USB2.0_16P, J3 Header, J6 47053-1000, J7 47053-1000, J8 SATA, J9 SATA, Q1 CSD18503Q5A, Q11 2N7002, Q12 2N7002, Q13 2N7002, Q2 CSD18504Q5A, Q3 CSD16321Q5, Q4 CSD16321Q5, Q5 2N7002, Q6 2N7002, Q7 2N7002, Q8 CSD17578Q5A, Q9 CSD17578Q5A, SW1 SW_Push, U1 LM5175RHF, U10 TLV75533PDBV, U2 LM5116MHX_NOPB, U3 TPS259803ONRGER, U4 TPS259804ONRGER, U5 TPS259804ONRGER, U6 TPS259803ONRGER, U7 STM32G431KBTx, U8 USBLC6-2SC6, U9 LT3080xST, Y1 ABM3B-8.000MHZ-10-D1G-T

Commit message: Rev 1.0 soft release (schematic is absolute dogshit)
Parts:
- added C83: 1nF, Capacitor_SMD:C_0805_2012Metric, F.Cu at (73.1, 90.8)
- added C84: 1nF, Capacitor_SMD:C_0805_2012Metric, B.Cu at (50.5, 80.7)
- added R75: 2.2R, Resistor_SMD:R_0805_2012Metric, F.Cu at (73.1, 88.8)
- added R76: 2.2R, Resistor_SMD:R_0805_2012Metric, B.Cu at (50.5, 82.7)
- C1: footprint Capacitor_SMD:C_0805_2012Metric -> Capacitor_SMD:C_0603_1608Metric
- C60: moved to B.Cu
- D12, D15, D16, D6, D7: value BAT54J -> BAT54WS
- moved NT2 9.19 mm to (51.0, 75.5), turned to 180 degrees
- moved R3 7.08 mm to (53.2, 75.5), turned to 180 degrees
- moved D12 3.47 mm to (105.8, 66.7), turned to 0 degrees
- moved D15 2.59 mm to (105.8, 68.6), turned to 180 degrees
- moved C60 2.59 mm to (63.2, 71.2)
- moved C51 0.74 mm to (77.7, 80.8)
- moved H2 0.71 mm to (142.0, 107.0)
- moved H3 0.71 mm to (29.0, 53.5)
- moved H4 0.71 mm to (29.0, 107.0)
- moved H1 0.50 mm to (127.0, 53.5)
- moved C1 0.45 mm to (64.7, 69.1)
- moved C50 0.14 mm to (77.7, 78.7)
Routing:
- net /PGOOD: track 15.3 -> 104.6 mm, vias 2 -> 4
- net /I_5V_SATA1: track 1.58 -> 66.6 mm, vias 0 -> 2
- net /12V_SATA1_PG: track 2.96 -> 64.1 mm, vias 1 -> 5
- net /5V_SATA1_PG: track 2.00 -> 58.1 mm, vias 1 -> 5
- net /I_5V_SATA2: track 1.58 -> 51.0 mm, vias 0 -> 2
- net /I_12V_SATA1: track 1.58 -> 48.8 mm, vias 0 -> 2
- net +12V: track 94.5 -> 140.3 mm, vias 31 -> 65
- net /5V_SATA2_PG: track 1.79 -> 46.2 mm, vias 1 -> 4
- net /I_12V_SATA2: track 0.00 -> 40.4 mm, vias 0 -> 2
- net /12V_SATA2_PG: track 2.46 -> 42.7 mm, vias 1 -> 5
- net +5V: track 40.9 -> 74.9 mm, vias 0 -> 2
- net /EN_A: track 127.7 -> 158.2 mm, vias 2 -> 3
- net /EN_B: track 135.9 -> 159.4 mm, vias 2 -> 4
- net +3.3V: track 13.7 -> 26.5 mm, vias 0 -> 10
- net 5175_VCC: track 10.9 -> 18.7 mm, vias 2 -> 3
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- added copper zone on In2.Cu, net +3.3V
- added copper zone on B.Cu, net GND
- added copper zone on F.Cu, net GND
- added copper zone on In2.Cu, net GND
Other:
- board text added: "lemp11 SATA Power Supply Rev 1.0 Alan Hsu"
