File: SATA_board/SATA_board.kicad_sch (KiCad schematic)
At the start: 5 parts, among them J1 47018-2001, J2 47018-2001, J3 678008025, J4 678008025, U1 LM5175RHF

Commit message: work
Parts:
- added J6, J7: 47053-1000, Connector:FanPinHeader_1x04_P2.54mm_Vertical, symbol Connector_Generic:Conn_01x04
Connections:
- net +3.3V_SATA1: now reaches J1.P1
- net +3.3V_SATA1: now also J1.P2, J1.P3
- net GND: now reaches J1.P10
- net GND: now also J1.P11, J1.P12, J1.P4, J1.P5, J1.P6, J1.SH1 (SHIELD), J1.SH2 (SHIELD), J2.P10, J2.P11, J2.P12, J2.P4, J2.P5, J2.P6, J2.SH1 (SHIELD), J2.SH2 (SHIELD), J6.1 (Pin_1), J7.1 (Pin_1)
- net +12V_SATA1: now reaches J1.P13
- net +12V_SATA1: now also J1.P14, J1.P15
- net +5V_SATA1: now reaches J1.P7
- net +5V_SATA1: now also J1.P8, J1.P9
- net at J1.S1: now also J3.1
- net at J1.S2: now also J3.2
- net at J1.S3: now also J3.3
- net at J1.S4: now also J3.4
- net at J1.S5: now also J3.5
- net at J1.S6: now also J3.6
- net at J1.S7: now also J3.7
- net +3.3V_SATA2: now reaches J2.P1
- net +3.3V_SATA2: now also J2.P2, J2.P3
- net +12V_SATA2: now reaches J2.P13
- net +12V_SATA2: now also J2.P14, J2.P15
- net +5V_SATA2: now reaches J2.P7
- net +5V_SATA2: now also J2.P8, J2.P9
- net at J2.S1: now also J4.1
- net at J2.S2: now also J4.2
- net at J2.S3: now also J4.3
- net at J2.S4: now also J4.4
- net at J2.S5: now also J4.5
- net at J2.S6: now also J4.6
- net at J2.S7: now also J4.7
- new net +12V: J6.2 (Pin_2), J7.2 (Pin_2)
- new net FAN1_PWM: J6.4 (Pin_4)
- new net FAN1_TACH: J6.3 (Pin_3)
- new net FAN2_PWM: J7.4 (Pin_4)
- new net FAN2_TACH: J7.3 (Pin_3)

Commit message: work
Parts:
- removed J1, J2: 47018-2001, 47018-2001:MOLEX_47018-2001, symbol 47018-2001:47018-2001
- removed J3, J4: 678008025, 678008025:CONN_67800-8025_MOL, symbol 678008025:678008025
- added C1, C14, C15, C6: 100nF, symbol Device:C
- added C10, C11, C8, C9: PCM1K680MCL1GS, Capacitor_SMD:CP_Elec_10x10, symbol Device:C_Polarized
- added C12, C13: 22uF, symbol Device:C
- added C16, C17, C18, C19, C20, C21, C22: 10uF, symbol Device:C
- added C2: 150pF, symbol Device:C
- added C3: 47pF, symbol Device:C
- added C4: 2.7nF, symbol Device:C
- added C5: 10pF, symbol Device:C
- added C7: 8nF, symbol Device:C
- added D1, D2, D3, D4, D5: D_Schottky, symbol Device:D_Schottky
- added J1: 105310-1204, Connector_Molex:Molex_Nano-Fit_105310-xx04_2x02_P2.50mm_Vertical, symbol Connector_Generic:Conn_02x02_Top_Bottom
- added J8, J9: SATA, Connector_Molex:Molex_Micro-Fit_3.0_43045-0612_2x03_P3.00mm_Vertical, symbol Connector_Generic:Conn_02x03_Top_Bottom
- added L1: 4.7uH, symbol Device:L
- added Q1, Q2, Q3, Q4: Si7336ADP, Package_SO:PowerPAK_SO-8_Single, symbol Transistor_FET:Si7336ADP
- added Q5, Q6: 2N7002, Package_TO_SOT_SMD:SOT-23, symbol Transistor_FET:2N7002
- added R1: 10R, symbol Device:R
- added R10, R9: 100R, symbol Device:R
- added R11, R13, R15: 100K, symbol Device:R
- added R12: 7.15K, symbol Device:R
- added R14: 1K, symbol Device:R
- added R2: 115K, symbol Device:R
- added R3: 8m, symbol Device:R
- added R4: 0R, symbol Device:R
- added R5: DNP, symbol Device:R
- added R6: 12.1K, symbol Device:R
- added R7: 200K, symbol Device:R
- added R8: 52.3K, symbol Device:R
Connections:
- net +12V: now also U1.10 (ISNS(-)), U1.11 (ISNS(+)), U1.21 (BIAS), U1.9 (VOSNS), C10.1, C11.1, C12.1, C13.1, C8.1, C9.1, D3.1 (K), Q3.5 (D), R11.1
- net +12V_SATA1: now also J8.1 (Pin_1)
- net +12V_SATA2: now also J9.1 (Pin_1)
- net +5V_SATA1: now also J8.2 (Pin_2), J8.5 (Pin_5)
- net +5V_SATA2: now also J9.2 (Pin_2), J9.5 (Pin_5)
- net GND: now also U1.19 (PGND), U1.29 (PowerPAD), U1.7 (AGND), C1.2, C10.2, C11.2, C12.2, C13.2, C16.2, C17.2, C18.2, C19.2, C2.2, C20.2, C21.2, C22.2, C4.2, C5.2, C6.2, C7.2, C8.2, C9.2, J1.2 (Pin_2), J1.4 (Pin_4), J8.4 (Pin_4), J8.6 (Pin_6), J9.4 (Pin_4), J9.6 (Pin_6), Q5.2 (S), Q6.2 (S), R12.2, R13.2, R2.2, R3.2, R4.2, R8.2, R9.2
- net 5175_MODE: now reaches U1.1 (MODE)
- net 5175_MODE: now also R4.1, R5.2
- net at U1.12 (CSG): now also C3.2, R9.1
- net at U1.13 (CS): now also C3.1, R10.1
- net ~{SHDN_OD}: now reaches U1.14 (PGOOD)
- net SW2: now reaches U1.15 (SW2)
- net SW2: now also C15.2, D3.2 (A), L1.2, Q3.1 (S), Q3.2 (S), Q3.3 (S), Q4.5 (D)
- net HDRV2: now reaches U1.16 (HDRV2)
- net HDRV2: now also Q3.4 (G)
- net BOOT2: now reaches U1.17 (BOOT2)
- net BOOT2: now also C15.1, D5.1 (K)
- net LDRV2: now reaches U1.18 (LDRV2)
- net LDRV2: now also Q4.4 (G)
- net 5175_DITH: now reaches U1.2 (DITH)
- net 5175_DITH: now also C7.1
- net 5175_VCC: now reaches U1.20 (VCC)
- net 5175_VCC: now also D4.2 (A), D5.2 (A), R5.1
- net LDRV1: now reaches U1.22 (LDRV1)
- net LDRV1: now also Q2.4 (G)
- net BOOT1: now reaches U1.23 (BOOT1)
- net BOOT1: now also C14.1, D4.1 (K)
- net HDRV1: now reaches U1.24 (HDRV1)
- net HDRV1: now also Q1.4 (G)
- net SW1: now reaches U1.25 (SW1)
- net SW1: now also C14.2, D2.1 (K), L1.1, Q1.1 (S), Q1.2 (S), Q1.3 (S), Q2.5 (D)
- net at U1.26 (EN/UVLO): now also Q5.3 (D), R7.2, R8.1
- net at U1.27 (VIN): now also C1.1, R1.2
- net VIN: now reaches U1.28 (VISNS)
- net VIN: now also C16.1, C17.1, C18.1, C19.1, C20.1, C21.1, C22.1, D1.2 (A), J1.1 (Pin_1), Q1.5 (D), R15.1, R7.1
- net 5175_RT: now reaches U1.3 (RT/SYNC)
- net 5175_RT: now also R2.1
- net 51751_SLOPE: now reaches U1.4 (SLOPE)
- net 51751_SLOPE: now also C2.1
- net 5175_SS: now reaches U1.5 (SS)
- net 5175_SS: now also C6.1
- net 5175_COMP: now reaches U1.6 (COMP)
- net 5175_COMP: now also C5.1, R6.1
- net FB: now reaches U1.8 (FB)
- net FB: now also R11.2, R12.1
- new net: Q6.1 (G), R13.1, R14.2
- new net: C4.1, R6.2
- new net: Q5.1 (G), Q6.3 (D), R15.2
- new net: D1.1 (K), R1.1
- new net 3V3_M2: J1.3 (Pin_3), R14.1
- new net CS: D2.2 (A), Q2.1 (S), Q2.2 (S), Q2.3 (S), Q4.1 (S), Q4.2 (S), Q4.3 (S), R10.2, R3.1
Other:
- note added: "Corsair Type 5 Cable"
- moved on the sheet: U1

Commit message: fix symbol
Parts:
- added U2, U3: TPS259802ONRGER, TPS259802:IC24_TPS259802ONRGER_TEX, symbol TPS259802:TPS259802ONRGER
Connections:
- net GND: now also U2.14 (GND), U2.4 (GND), U2.5 (GND), U3.14 (GND), U3.4 (GND), U3.5 (GND)
- new net: U2.17 (OUT), U2.18 (OUT), U2.19 (OUT), U2.20 (OUT), U2.21 (OUT), U2.22 (OUT), U2.23 (OUT), U2.24 (OUT)
- new net: U3.17 (OUT), U3.18 (OUT), U3.19 (OUT), U3.20 (OUT), U3.21 (OUT), U3.22 (OUT), U3.23 (OUT), U3.24 (OUT)
- new net IN: U2.16 (IN), U2.2 (IN), U2.3 (IN), U3.16 (IN), U3.2 (IN), U3.3 (IN)

Commit message: continued schematic work
Parts:
- removed D1, D2, D3, D4, D5: D_Schottky, symbol Device:D_Schottky
- removed Q1, Q2, Q3, Q4: Si7336ADP, Package_SO:PowerPAK_SO-8_Single, symbol Transistor_FET:Si7336ADP
- removed U2, U3: TPS259802ONRGER, TPS259802:IC24_TPS259802ONRGER_TEX, symbol TPS259802:TPS259802ONRGER
- added C23, C27, C35, C45, C46: 1nF, symbol Device:C
- added C24, C25, C33, C34, C41, C42, C43, C44: 2.2nF, symbol Device:C
- added C26, C31, C37, C38: 4.7nF, symbol Device:C
- added C28, C29, C32, C39, C40, C54, C55, C56, C57: 22uF, symbol Device:C
- added C30, C36, C47, C48, C49, C58, C59, C60: 1uF, symbol Device:C
- added C50: 120pF, symbol Device:C
- added C51, C67, C68, C69, C70: 100nF, symbol Device:C
- added C52: 2.2uF, symbol Device:C
- added C53: 10uF, symbol Device:C
- added C61: PCM1K680MCL1GS, Capacitor_SMD:CP_Elec_10x10, symbol Device:C_Polarized
- added C62: 10nF, symbol Device:C
- added C63: 100pF, symbol Device:C
- added C64, C65: 12pF, Capacitor_SMD:C_0402_1005Metric, symbol Device:C
- added C66: 4.7uF, symbol Device:C
- added D1: SMAJ24A, Diode_SMD:D_SMA, symbol Diode:SMAJ24A
- added D10, D4, D5, D8: PMEG4010CEJ, Diode_SMD:D_SOD-323F, symbol Diode:PMEG4010CEJ
- added D13: BAT54C, Package_TO_SOT_SMD:SOT-23, symbol Diode:BAT54C
- added D2, D3: PMEG045T100EPD, Package_TO_SOT_SMD:Nexperia_CFP15_SOT-1289, symbol Diode:PMEG045T100EPD
- added D6, D7: BAT54J, Diode_SMD:D_SOD-323F, symbol Diode:BAT54J
- added D9: BZV55B10, Diode_SMD:D_MiniMELF, symbol Diode:BZV55B10
- added F1: Fuse, Fuse:Fuse_2512_6332Metric, symbol Device:Fuse
- added L2: 3.3uH, symbol Device:L
- added NT1, NT2: (no value), symbol Device:NetTie_2
- added Q1: CSD18503Q5A, Package_TO_SOT_SMD:TDSON-8-1, symbol Transistor_FET:CSD18503Q5A
- added Q2: CSD18504Q5A, Package_TO_SOT_SMD:TDSON-8-1, symbol Transistor_FET:CSD18504Q5A
- added Q3, Q4: CSD16321Q5, Package_TO_SOT_SMD:TDSON-8-1, symbol Transistor_FET:CSD16321Q5
- added Q8, Q9: CSD17578Q5A, Package_TO_SOT_SMD:TDSON-8-1, symbol Transistor_FET:CSD17578Q5A
- added R16, R24, R26, R27: 499R, symbol Device:R
- added R17, R20, R21, R25, R28, R29: 1K, symbol Device:R
- added R18, R23: 200K, symbol Device:R
- added R19, R22: 806K, symbol Device:R
- added R30, R32, R39: 100K, symbol Device:R
- added R31: 13K, symbol Device:R
- added R33: 5.6K, symbol Device:R
- added R34: 0R, symbol Device:R
- added R35: 13m, symbol Device:R
- added R36: 3.57K, symbol Device:R
- added R37: 1.15K, symbol Device:R
- added R38: 6.65K, symbol Device:R
- added R40: 10.5K, symbol Device:R
- added R41: 1.5K, symbol Device:R
- added R42, R43, R44, R45, R46: 10K, symbol Device:R
- added SW1: SW_Push, Button_Switch_THT:SW_PUSH_6mm, symbol Switch:SW_Push
- added U2: LM5116MHX_NOPB, LM5116MHX_NOPB:SOP65P640X110-21N, symbol LM5116MHX_NOPB:LM5116MHX_NOPB
- added U3, U6: TPS259803ONRGER, TPS259802:IC24_TPS259802ONRGER_TEX, symbol TPS259802:TPS259803ONRGER
- added U4, U5: TPS259804ONRGER, TPS259802:IC24_TPS259802ONRGER_TEX, symbol TPS259802:TPS259804ONRGER
- added U7: STM32G431KBTx, Package_QFP:LQFP-32_7x7mm_P0.8mm, symbol MCU_ST_STM32G4:STM32G431KBTx
- added Y1: ABM3B-8.000MHZ-10-D1G-T, 0_PAY_Footprint_Library:Crystal_SMD_Abracon_ABM3B-4Pin_5.0x3.2mm, symbol Device:Crystal_GND24
- C14, C15: value 100nF -> 470nF
- C4: value 2.7nF -> 3.9nF
- C5: value 10pF -> 220pF
- C7: value 8nF -> 8.2nF
- R1: value 10R -> 2.2R
- R6: value 12.1K -> 8.06K
Connections:
- net +12V: now also C29.1, C32.1, C53.1, D3.3 (K), D6.1 (K), D7.1 (K), Q3.5 (D), Q8.5 (D), R19.1, R22.1, R30.1, R32.1, U2.1 (VIN), U2.17 (VCCX), U4.25 (PAD_IN), U4.[1-3,16] (IN), U5.25 (PAD_IN), U5.[1-3,16] (IN)
- net +12V_SATA1: now also C30.1, U4.[17-24] (OUT)
- net +12V_SATA2: now also C36.1, U5.[17-24] (OUT)
- net +5V_SATA1: now also C47.1, U3.[17-24] (OUT)
- net +5V_SATA2: now also C48.1, U6.[17-24] (OUT)
- net 5175_VCC: now also C60.1, D4.2 (A), D5.2 (A)
- net BOOT1: now also D4.1 (K)
- net BOOT2: now also D5.1 (K)
- net CS: now also D2.1 (A), D2.2 (A), Q2.1 (S), Q2.2 (S), Q2.3 (S), Q4.1 (S), Q4.2 (S), Q4.3 (S)
- net FAN1_PWM: now also U7.25 (PA15)
- net FAN1_TACH: now also U7.27 (PB4)
- net FAN2_PWM: now also U7.26 (PB3)
- net FAN2_TACH: now also U7.28 (PB5)
- net GND: now also C23.2, C24.2, C25.2, C26.2, C27.2, C28.2, C29.2, C30.2, C31.2, C32.2, C33.2, C34.2, C35.2, C36.2, C37.2, C38.2, C39.2, C40.2, C41.2, C42.2, C43.2, C44.2, C45.2, C46.2, C47.2, C48.2, C49.2, C50.2, C51.2, C52.2, C53.2, C54.2, C55.2, C56.2, C57.2, C58.2, C60.2, C61.2, C64.1, C65.1, C66.2, C67.2, C68.2, C69.2, C70.2, D1.2 (A2), D9.2 (A), NT1.2, NT2.2, R16.2, R17.2, R18.2, R23.2, R24.2, R25.2, R26.2, R27.2, R28.2, R29.2, R31.2, R33.2, R34.2, R35.2, R37.2, R41.2, SW1.1, U2.14 (PGND), U2.21 (EXP), U2.6 (AGND), U3.12 (LDSTRT), U3.14 (GND), U3.26 (PAD_GND), U3.4 (GND), U3.5 (GND), U4.12 (LDSTRT), U4.14 (GND), U4.26 (PAD_GND), U4.4 (GND), U4.5 (GND), U5.12 (LDSTRT), U5.14 (GND), U5.26 (PAD_GND), U5.4 (GND), U5.5 (GND), U6.12 (LDSTRT), U6.14 (GND), U6.26 (PAD_GND), U6.4 (GND), U6.5 (GND), U7.14 (VSSA), U7.16 (VSS), U7.32 (VSS), Y1.2 (G), Y1.4 (G); no longer R9.2
- net HDRV1: now also Q1.4 (G)
- net HDRV2: now also Q3.4 (G)
- net LDRV1: now also Q2.4 (G)
- net LDRV2: now also Q4.4 (G)
- net SW1: now also D2.3 (K), Q1.1 (S), Q1.2 (S), Q1.3 (S), Q2.5 (D)
- net SW2: now also D3.1 (A), D3.2 (A), Q3.1 (S), Q3.2 (S), Q3.3 (S), Q4.5 (D)
- net VIN: now also F1.1; no longer C16.1, C17.1, C18.1, C19.1, C20.1, C21.1, C22.1, U1.28 (VISNS)
- net at Q5.1 (G), Q6.3 (D), R15.2: now also D9.1 (K)
- net at R1.1: now also D10.1 (K)
- net ~{SHDN_OD} renamed PGOOD
- net PGOOD: now also D13.3, R46.2, U7.18 (PA8)
- new net: D13.1, R20.1
- new net: C59.2, L2.1, Q8.1 (S), Q8.2 (S), Q8.3 (S), Q9.5 (D), U2.20 (SW)
- new net: Q8.4 (G), U2.19 (HO)
- new net: C63.2, R36.2, R37.1, R38.1, U2.8 (FB)
- new net: C62.1, R38.2
- new net: C49.1, R30.2, R31.1, U2.2 (UVLO)
- new net: C37.1, U3.7 (ITIMER)
- new net: C59.1, D8.1 (K), U2.18 (HB)
- new net: C25.1, U4.11 (NRETRY)
- new net: D13.2, R21.1
- new net: R39.2, SW1.2, U7.4 (PG10)
- new net: C45.1, U3.15 (dVdt)
- new net: C31.1, U5.7 (ITIMER)
- new net: C24.1, U4.10 (RETRY_DLY)
- new net: C50.1, U2.5 (RAMP)
- new net: C64.2, U7.2 (PF0), Y1.3
- new net: C65.2, U7.3 (PF1), Y1.1
- new net: R16.1, U4.8 (ILIM)
- new net: C62.2, C63.1, U2.9 (COMP)
- new net: NT1.1, U2.13 (CSG)
- new net: C42.1, U6.10 (RETRY_DLY)
- new net: C34.1, U5.11 (NRETRY)
- new net: R33.1, U2.3 (RT/SYNC)
- new net: C33.1, U5.10 (RETRY_DLY)
- new net: R26.1, U3.8 (ILIM)
- new net: C35.1, U5.15 (dVdt)
- new net: C23.1, U4.15 (dVdt)
- new net: C26.1, U4.7 (ITIMER)
- new net: C44.1, U6.11 (NRETRY)
- new net: C46.1, U6.15 (dVdt)
- new net: C38.1, U6.7 (ITIMER)
- new net: R27.1, U6.8 (ILIM)
- new net: C51.1, U2.7 (SS)
- new net: Q9.1 (S), Q9.2 (S), Q9.3 (S), R35.1, U2.12 (CS)
- new net: C43.1, U3.11 (NRETRY)
- new net: R34.1, U2.11 (DEMB)
- new net: Q9.4 (G), U2.15 (LO)
- new net: R32.2, U2.4 (EN)
- new net: C41.1, U3.10 (RETRY_DLY)
- new net: R24.1, U5.8 (ILIM)
- new net +3.3V: C66.1, C67.1, C68.1, C69.1, R39.1, R42.1, R43.1, R44.1, R45.1, R46.1, U7.1 (VDD), U7.15 (VDDA), U7.17 (VDD)
- new net +5V: C39.1, C40.1, C54.1, C55.1, C56.1, C57.1, C58.1, L2.2, R36.1, U2.10 (VOUT), U3.25 (PAD_IN), U3.[1-3,16] (IN), U6.25 (PAD_IN), U6.[1-3,16] (IN)
- new net 12V_SATA1_PG: R42.2, U4.13 (PG), U7.9 (PA4)
- new net 12V_SATA2_PG: R43.2, U5.13 (PG), U7.10 (PA5)
- new net 5116_VCC: C52.1, D8.2 (A), U2.16 (VCC)
- new net 5V_SATA1_PG: R44.2, U3.13 (PG), U7.11 (PA6)
- new net 5V_SATA2_PG: R45.2, U6.13 (PG), U7.12 (PA7)
- new net CSG: NT2.1, R9.2
- new net EN_A: C27.1, D6.2 (A), R18.1, R19.2, R20.2, U3.6 (EN/UVLO), U4.6 (EN/UVLO)
- new net EN_B: C28.1, D7.2 (A), R21.2, R22.2, R23.1, U5.6 (EN/UVLO), U6.6 (EN/UVLO)
- new net I_12V_SATA1: R17.1, U4.9 (IMON), U7.5 (PA0)
- new net I_12V_SATA2: R25.1, U5.9 (IMON), U7.7 (PA2)
- new net I_5V_SATA1: R28.1, U3.9 (IMON), U7.6 (PA1)
- new net I_5V_SATA2: R29.1, U6.9 (IMON), U7.8 (PA3)
- new net SWCLK: U7.24 (PA14)
- new net SWDIO: U7.23 (PA13)
- new net VIN_ADC: C70.1, R40.2, R41.1, U7.13 (PB0)
- new net VIN_F: C16.1, C17.1, C18.1, C19.1, C20.1, C21.1, C22.1, C61.1, D1.1 (A1), D10.2 (A), F1.2, Q1.5 (D), R40.1, U1.28 (VISNS)
Other:
- note added: "91.7ms retry delay, 4 retries"
- note added: "~3A nominal fast trip limit"
- moved on the sheet: C1, C10, C11, C12, C13, C14, C15, C16, C17, C18, C19, C2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

Commit message: complete schematic, but it looks absolutely awful
Parts:
- removed J1: 105310-1204, Connector_Molex:Molex_Nano-Fit_105310-xx04_2x02_P2.50mm_Vertical, symbol Connector_Generic:Conn_02x02_Top_Bottom
- added C71: 10uF, Capacitor_SMD:C_1210_3225Metric, symbol Device:C
- added C72, C74, C79, C80, C81, C82: 10uF, Capacitor_SMD:C_0805_2012Metric, symbol Device:C
- added C73, C75, C76, C77, C78: 100nF, Capacitor_SMD:C_0603_1608Metric, symbol Device:C
- added D11: SMF6V0A, Diode_SMD:D_SMF, symbol Diode:SMF6V0A
- added D12, D15, D16: BAT54J, Diode_SMD:D_SOD-323F, symbol Diode:BAT54J
- added D14: BAT54C, Package_TO_SOT_SMD:SOT-23, symbol Diode:BAT54C
- added H1, H2, H3, H4: M3, MountingHole:MountingHole_3.2mm_M3_DIN965_Pad, symbol Mechanical:MountingHole_Pad
- added J1: 105310-1206, Connector_Molex:Molex_Nano-Fit_105310-xx06_2x03_P2.50mm_Vertical, symbol Connector_Generic:Conn_02x03_Top_Bottom
- added J2: USB_C_Receptacle_USB2.0_16P, Connector_USB:USB_C_Receptacle_GCT_USB4105-xx-A_16P_TopMnt_Horizontal, symbol Connector:USB_C_Receptacle_USB2.0_16P
- added J3: Header, Connector_PinHeader_2.54mm:PinHeader_2x03_P2.54mm_Vertical, symbol Connector_Generic:Conn_02x03_Odd_Even
- added Q11, Q12, Q13, Q7: 2N7002, Package_TO_SOT_SMD:SOT-23, symbol Transistor_FET:2N7002
- added R47, R48: 10R, Resistor_SMD:R_0402_1005Metric, symbol Device:R
- added R49, R50: 5.1K, Resistor_SMD:R_0402_1005Metric, symbol Device:R
- added R51, R52, R53, R60, R61, R66, R68: 100R, Resistor_SMD:R_0603_1608Metric, symbol Device:R
- added R54: 430K, Resistor_SMD:R_0603_1608Metric, symbol Device:R
- added R55, R56, R57, R58, R59, R62, R63, R64, R65, R67, R69: 10K, Resistor_SMD:R_0603_1608Metric, symbol Device:R
- added R70: 8.2K, Resistor_SMD:R_0603_1608Metric, symbol Device:R
- added R71, R72, R73, R74: 3.3R, Resistor_SMD:R_0402_1005Metric, symbol Device:R
- added U10: TLV75533PDBV, Package_TO_SOT_SMD:SOT-23-5, symbol Regulator_Linear:TLV75533PDBV
- added U8: USBLC6-2SC6, Package_TO_SOT_SMD:SOT-23-6, symbol Power_Protection:USBLC6-2SC6
- added U9: LT3080xST, Package_TO_SOT_SMD:SOT-223, symbol Regulator_Linear:LT3080xST
- C1: footprint (none) -> Capacitor_SMD:C_0805_2012Metric
- C12, C13, C16, C17, C18, C19, C20, C21, C22, C53, C54, C55, C56, C57: footprint (none) -> Capacitor_SMD:C_1210_3225Metric
- C14, C15, C23, C24, C25, C26, C27, C30, C31, C33, C34, C35, C36, C37, C38, C41, C42, C43, C44, C45, C46, C47, C48, C49, C50, C51, C52, C58, C59, C60, C62, C63, C66, C67, C68, C69, C70: footprint (none) -> Capacitor_SMD:C_0603_1608Metric
- C2, C3, C4, C5, C6, C7: footprint (none) -> Capacitor_SMD:C_0402_1005Metric
- C28: value 22uF -> 100uF; footprint (none) -> Capacitor_SMD:C_1210_3225Metric
- C29, C32, C39, C40: value 22uF -> 10uF; footprint (none) -> Capacitor_SMD:C_0805_2012Metric
- F1: value Fuse -> SF-1206S1000W-2; footprint Fuse:Fuse_2512_6332Metric -> Fuse:Fuse_1206_3216Metric
- L1: footprint (none) -> Inductor_SMD:L_Vishay_IHLP-6767; PN (none) -> IHLP6767GZER4R7M01
- L2: footprint (none) -> Inductor_SMD:L_Vishay_IHLP-4040; PN (none) -> IHLP4040DZER3R3M01
- NT1, NT2: footprint (none) -> NetTie:NetTie-2_SMD_Pad0.5mm
- R1, R11, R12, R13, R14, R15, R16, R18, R19, R20, R21, R22, R23, R24, R26, R27, R30, R31, R32, R33, R34, R36, R37, R38, R39, R40, R41, R42, R43, R44, R45, R46, R7, R8: footprint (none) -> Resistor_SMD:R_0603_1608Metric
- R10, R2, R4, R6, R9: footprint (none) -> Resistor_SMD:R_0402_1005Metric
- R17, R25, R28, R29: value 1K -> 1.5K; footprint (none) -> Resistor_SMD:R_0603_1608Metric
- R3, R35: footprint (none) -> Resistor_SMD:R_2512_6332Metric
- R5: value DNP -> 0R; footprint (none) -> Resistor_SMD:R_0402_1005Metric; now not fitted
- U2: footprint LM5116MHX_NOPB:SOP65P640X110-21N -> LM5116:SOP65P640X110-21N
- Y1: footprint 0_PAY_Footprint_Library:Crystal_SMD_Abracon_ABM3B-4Pin_5.0x3.2mm -> Crystal:Crystal_SMD_Abracon_ABM3B-4Pin_5.0x3.2mm
Connections:
- net +12V: now also C81.1, C82.1
- net +3.3V: now also C80.1, D12.1 (K), J3.1 (Pin_1), R58.1, R59.1, U10.5 (OUT), U8.5 (VBUS)
- net +5V: now also D16.2 (A)
- net 3V3_M2: now also J1.6 (Pin_6)
- net FAN1_PWM: now also R60.2; no longer J6.4 (Pin_4)
- net FAN1_TACH: now also R59.2
- net FAN2_PWM: now also R61.2; no longer J7.4 (Pin_4)
- net FAN2_TACH: now also R58.2
- net GND: now also U7.20 (PA10), C71.2, C72.2, C73.2, C74.2, C75.2, C76.2, C77.2, C78.2, C79.2, C80.2, C81.2, C82.2, D11.2 (A2), D15.2 (A), H1.1, H2.1, H3.1, H4.1, J1.3 (Pin_3), J1.4 (Pin_4), J1.5 (Pin_5), J2.A1 (GND), J2.A12 (GND), J2.B1 (GND), J2.B12 (GND), J2.SH (SHIELD), J3.5 (Pin_5), J3.6 (Pin_6), Q11.2 (S), Q12.2 (S), Q13.2 (S), Q7.2 (S), R49.1, R50.1, R54.2, R56.2, R62.2, R65.2, R67.2, R69.2, R70.2, U10.2 (GND), U8.2 (GND)
- net HDRV1: now also R74.1; no longer Q1.4 (G)
- net HDRV2: now also R71.1; no longer Q3.4 (G)
- net I_12V_SATA1: now also C76.1, R57.2; no longer R17.1, U4.9 (IMON)
- net I_12V_SATA2: now also C78.1, R64.2; no longer R25.1, U5.9 (IMON)
- net I_5V_SATA1: now also C77.1, R63.2; no longer R28.1, U3.9 (IMON)
- net I_5V_SATA2: now also C75.1, R55.2; no longer R29.1, U6.9 (IMON)
- net LDRV1: now also R73.1; no longer Q2.4 (G)
- net LDRV2: now also R72.1; no longer Q4.4 (G)
- net SWCLK: now also R52.1
- net SWDIO: now also R51.1
- net VIN: now also J1.1 (Pin_1), J1.2 (Pin_2); no longer R15.1, R7.1
- net VIN_ADC: now also D12.2 (A), D15.1 (K)
- net VIN_F: now also R15.1, R7.1, C71.1, U9.3 (IN)
- net at D13.1, R20.1: now also Q13.3 (D)
- net at D13.2, R21.1: now also Q12.3 (D)
- net nRST: now reaches R39.2, SW1.2, U7.4 (PG10)
- net nRST: now also C73.1, R53.1
- net USB_D-: now reaches U7.21 (PA11)
- net USB_D-: now also R47.2
- net USB_D+: now reaches U7.22 (PA12)
- net USB_D+: now also R48.2
- net DIS_A: now reaches U7.29 (PB6)
- net DIS_A: now also R68.2
- net DIS_B: now reaches U7.30 (PB7)
- net DIS_B: now also R66.2
- net at U7.31 (PB8): now also R65.1
- new net: Q7.1 (G), R56.1, R60.1
- new net: J6.4 (Pin_4), Q7.3 (D)
- new net: R25.1, R64.1, U5.9 (IMON)
- new net: J3.2 (Pin_2), R51.2
- new net: Q12.1 (G), R66.1, R67.1
- new net: Q11.1 (G), R61.1, R62.1
- new net: J7.4 (Pin_4), Q11.3 (D)
- new net: C79.1, D14.3, D16.1 (K), U10.1 (IN), U10.3 (EN)
- new net: R47.1, U8.6 (I/O1)
- new net: Q13.1 (G), R68.1, R69.1
- new net: J2.B5 (CC2), R50.2
- new net: J3.3 (Pin_3), R53.2
- new net: R29.1, R55.1, U6.9 (IMON)
- new net: Q1.4 (G), R74.2
- new net: R17.1, R57.1, U4.9 (IMON)
- new net: Q2.4 (G), R73.2
- new net: Q3.4 (G), R71.2
- new net: R54.1, U9.1 (SET)
- new net: J3.4 (Pin_4), R52.2
- new net: R28.1, R63.1, U3.9 (IMON)
- new net: J2.A5 (CC1), R49.2
- new net: J2.A6 (D+), J2.B6 (D+), U8.3 (I/O2)
- new net: J2.A7 (D-), J2.B7 (D-), U8.1 (I/O1)
- new net: R48.1, U8.4 (I/O2)
- new net: Q4.4 (G), R72.2
- new net 4V3_STBY: C72.1, D14.2, R70.1, U9.2 (OUT), U9.4 (OUT)
- new net 5V_USB: C74.1, D11.1 (A1), D14.1, J2.A4 (VBUS), J2.A9 (VBUS), J2.B4 (VBUS), J2.B9 (VBUS)
Other:
- moved on the sheet: C27, C28, C70, D13, D6, D7, J6, J7, R16, R18, R19, R20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

Commit message: Rev 1.0 soft release (schematic is absolute dogshit)
Parts:
- added C83, C84: 1nF, Capacitor_SMD:C_0805_2012Metric, symbol Device:C
- added R75, R76: 2.2R, Resistor_SMD:R_0805_2012Metric, symbol Device:R
- C1: footprint Capacitor_SMD:C_0805_2012Metric -> Capacitor_SMD:C_0603_1608Metric; MP (none) -> C0603C104K5RACTU
- C10, C11, C61, C8, C9: MP (none) -> PCM1K680MCL1GS
- C12, C13, C54, C55, C56, C57: MP (none) -> CGA6P3X7R1E226M250AB
- C14, C15: MP (none) -> GRM188R71E474KA12J
- C16, C17, C18, C19, C20, C21, C22, C53, C71: MP (none) -> CL32B106KMVNNWE
- C2: MP (none) -> GRM1555C1H151JA01D
- C23, C27, C35, C45, C46: MP (none) -> CL10B102KB8NNNC
- C24, C25, C33, C34, C41, C42, C43, C44: MP (none) -> C0603C222K5RACTU
- C26, C31, C37, C38: MP (none) -> CL10B472KB8NNNC
- C28: MP (none) -> GRM32EC70J107ME15L
- C29, C32, C39, C40, C72, C74, C79, C80, C81, C82: MP (none) -> GMC21X7R106K25NT
- C3: MP (none) -> CC0402JRNPO9BN470
- C30, C36, C47, C48, C49, C58, C59, C60: MP (none) -> TMK107B7105MA-T
- C4: MP (none) -> GRM1555C1H392JE01D
- C5: MP (none) -> GRM1555C1H221JA01D
- C50: MP (none) -> CL10C121JB8NNNC
- C51, C67, C68, C69, C70, C73, C75, C76, C77, C78: MP (none) -> C0603C104K5RACTU
- C52: MP (none) -> GRM188Z71E225ME43D
- C6: MP (none) -> GRM155R71H104KE14D
- C62: MP (none) -> CL10B103KA8WPNC
- C63: MP (none) -> CL10C101JB8NNNC
- C64, C65: MP (none) -> GCM1555C1H120FA16D
- C66: MP (none) -> KAM15CR70J475MT
- C7: MP (none) -> GCM155R71H822KA55D
- D1: MP (none) -> SMAJ24A
- D10, D4, D5, D8: MP (none) -> PMEG4010CEJ
- D11: MP (none) -> SMF6V0A
- D12, D15, D16, D6, D7: value BAT54J -> BAT54WS; MP (none) -> BAT54WS
- D13, D14: MP (none) -> BAT54C
- D2, D3: MP (none) -> PMEG045T100EPD
- D9: MP (none) -> BZV55B10
- F1: MP (none) -> SF-1206S1000W-2
- J1: MP (none) -> 105310-1206
- J2: MP (none) -> USB4105-GF-A-120
- J3: MP (none) -> M20-9980346
- J6, J7: MP (none) -> 47053-1000
- J8, J9: MP (none) -> 43045-0612
- L1: MP (none) -> IHLP6767GZER4R7M01; PN IHLP6767GZER4R7M01 -> (none)
- L2: MP (none) -> IHLP4040DZER3R3M01; PN IHLP4040DZER3R3M01 -> (none)
- Q1: MP (none) -> CSD18503Q5A
- Q11, Q12, Q13, Q5, Q6, Q7: MP (none) -> 2N7002
- Q2: MP (none) -> CSD18504Q5A
- Q3, Q4: MP (none) -> CSD16321Q5
- Q8, Q9: MP (none) -> CSD17578Q5A
- R1: MP (none) -> ERJ-3GEYJ2R2V
- R10, R9: MP (none) -> RC0402FR-07100RL
- R11, R13, R15, R30, R32, R39: MP (none) -> CRCW0603100KFKEA
- R12: MP (none) -> RMCF0603FT7K15
- R14, R20, R21: MP (none) -> ERJ-3RBD102V
- R16, R24, R26, R27: MP (none) -> RC0603FR-07499RL
- R17, R25, R28, R29, R41: MP (none) -> RC0603FR-071K5L
- R18, R23, R7: MP (none) -> ERJ-3EKF2003V
- R19, R22: MP (none) -> CRCW0603806KFKEA
- R2: MP (none) -> CR0402-FX-1153GLF
- R3: MP (none) -> CRF2512-FZ-R008ELF
- R31: MP (none) -> RC0603FR-0713KL
- R33: MP (none) -> RK73H1JTTD5601F
- R34: MP (none) -> RC0603JR-070RL
- R35: MP (none) -> WPC2512QLR013FYR
- R36: MP (none) -> RMCF0603FT3K57
- R37: MP (none) -> RC0603FR-071K15L
- R38: MP (none) -> RC0603FR-076K65L
- R4, R5: MP (none) -> RC0402JR-070RP
- R40: MP (none) -> RC0603FR-0710K5L
- R42, R43, R44, R45, R46, R55, R56, R57, R58, R59, R62, R63, R64, R65, R67, R69: MP (none) -> CRCW060310K0FKEA
- R47, R48: MP (none) -> RC0402FR-0710RL
- R49, R50: MP (none) -> RC0402FR-075K1L
- R51, R52, R53, R60, R61, R66, R68: MP (none) -> ERJ-3EKF1000V
- R54: MP (none) -> RK73H1JTTD4303F
- R6: MP (none) -> CRCW04028K06FKED
- R70: MP (none) -> RC0603FR-078K2L
- R71, R72, R73, R74: MP (none) -> RC0402FR-133R3L
- R8: MP (none) -> RMCF0603FT52K3
- SW1: MP (none) -> B3F-1000
- U1: MP (none) -> LM5175RHFR
- U10: MP (none) -> TLV75533PDBV
- U2: MP LM5116MHX -> LM5116MH/NOPB
- U3, U6: MP (none) -> TPS259803ONRGER
- U4, U5: MP (none) -> TPS259804ONRGER
- U7: MP (none) -> STM32G431KBT6
- U8: MP (none) -> USBLC6-2SC6
- U9: MP (none) -> LT3080EST#TRPBF
- Y1: MP (none) -> ABM3B-8.000MHZ-10-D1G-T
Connections:
- net GND: now also C83.2, C84.2
- net SW1: now also R76.1
- net SW2: now also R75.1
- new net: C83.1, R75.2
- new net: C84.1, R76.2
